File: pcb/pcb-oven-controller.kicad_pcb (KiCad board)
At the start: 4 copper layers, 30 x 25 mm, 17 parts, among them J1 USB_A, SW1 SW_Push, U1 STM32F411CEUx, Y1 25Mhz

Commit message: Add more pcb progress
Parts:
- added C11: 100nF, Capacitor_SMD:C_0603_1608Metric, F.Cu at (68.6, 92.4)
- added C12: 100nF, Capacitor_SMD:C_0402_1005Metric, F.Cu at (88.9, 98.4)
- added C12: 100nF, Capacitor_SMD:C_0402_1005Metric, F.Cu at (89.0, 68.5)
- added C13: 10nF, Capacitor_SMD:C_0603_1608Metric, F.Cu at (142.0, 117.3)
- added C14: 10nF, Capacitor_SMD:C_0603_1608Metric, F.Cu at (68.6, 97.4)
- added C15: 10nF, Capacitor_SMD:C_0603_1608Metric, F.Cu at (88.0, 57.5)
- added C16: 10nF, Capacitor_SMD:C_0603_1608Metric, B.Cu at (132.2, 99.2)
- added C17: 10uF, Capacitor_SMD:C_0603_1608Metric, F.Cu at (79.3, 66.3)
- added C18: 100nF, Capacitor_SMD:C_0402_1005Metric, F.Cu at (82.8, 73.1)
- added C19: 100nF, Capacitor_SMD:C_0603_1608Metric, F.Cu at (144.7, 121.0)
- added C20: 100nF, Capacitor_SMD:C_0603_1608Metric, F.Cu at (81.7, 119.5)
- added FB1: 100R, Inductor_SMD:L_0603_1608Metric, F.Cu at (89.6, 66.3)
- added J3: TC2030, Connector:Tag-Connect_TC2030-IDC-NL_2x03_P1.27mm_Vertical, F.Cu at (125.0, 79.2)
- added R10: 4.7k, Resistor_SMD:R_0603_1608Metric, F.Cu at (72.6, 102.4)
- added R11: 4.7k, Resistor_SMD:R_0603_1608Metric_Pad0.98x0.95mm_HandSolder, F.Cu at (85.2, 92.4)
- added R12: 4.7k, Resistor_SMD:R_0603_1608Metric_Pad0.98x0.95mm_HandSolder, F.Cu at (140.0, 95.6)
- added R13: 4.7k, Resistor_SMD:R_0603_1608Metric_Pad0.98x0.95mm_HandSolder, F.Cu at (140.0, 99.4)
- added R14: 4.7k, Resistor_SMD:R_0603_1608Metric, F.Cu at (79.3, 68.8)
- added R15: 4.7k, Resistor_SMD:R_0603_1608Metric, F.Cu at (79.3, 71.3)
- added R3: 50k, Resistor_SMD:R_0603_1608Metric, F.Cu at (68.6, 99.9)
- added R4: 50k, Resistor_SMD:R_0603_1608Metric, F.Cu at (68.6, 102.4)
- added R5: 270k, Resistor_SMD:R_0603_1608Metric, F.Cu at (68.6, 104.9)
- added R6: 50k, Resistor_SMD:R_0603_1608Metric, F.Cu at (72.6, 92.4)
- added R7: 50k, Resistor_SMD:R_0603_1608Metric, F.Cu at (72.6, 94.9)
- added R8: 4.7k, Resistor_SMD:R_0603_1608Metric, F.Cu at (72.6, 97.4)
- added R9: 4.7k, Resistor_SMD:R_0603_1608Metric, F.Cu at (72.6, 99.9)
- added TC1: Thermocouple_0, ATL:K_Thermocouple_Generic, F.Cu at (130.0, 112.0)
- added TC2: Thermocouple_1, ATL:K_Thermocouple_Generic, F.Cu at (129.8, 130.6)
- added U2: PCAL6416, Package_DFN_QFN:WQFN-24-1EP_4x4mm_P0.5mm_EP2.45x2.45mm, F.Cu at (144.4, 96.1)
- added U3: MAX31855KASA, Package_SO:SOIC-8_3.9x4.9mm_P1.27mm, F.Cu at (147.0, 117.5)
- added U4: MAX31855KASA, Package_SO:SOIC-8_3.9x4.9mm_P1.27mm, F.Cu at (78.8, 100.8)
- added U5: TMP1075DSG, Package_SON:WSON-8-1EP_2x2mm_P0.5mm_EP0.9x1.6mm_ThermalVias, F.Cu at (85.0, 57.6)
- added U6: TMP1075DSG, Package_SON:WSON-8-1EP_2x2mm_P0.5mm_EP0.9x1.6mm_ThermalVias, B.Cu at (135.2, 98.9)
Connections:
- net VDDA renamed +3.3VA
- FB1 pad 1: VDD -> +3.3V
- J1 pad 4: unconnected-(J1-Pad4) -> GND
- U1 pad 1: VDD -> +3.3V
- U1 pad 16: unconnected-(U1-Pad16) -> SDIO_CMD
- U1 pad 24: VDD -> +3.3V
- U1 pad 28: unconnected-(U1-Pad28) -> SDIO_CK
- U1 pad 34: unconnected-(U1-Pad34) -> SWDIO
- U1 pad 36: VDD -> +3.3V
- U1 pad 37: unconnected-(U1-Pad37) -> SWCLK
- U1 pad 39: unconnected-(U1-Pad39) -> SWO
- U1 pad 41: unconnected-(U1-Pad41) -> SDIO_CD
- U1 pad 43: unconnected-(U1-Pad43) -> SDIO_D0
- U1 pad 45: unconnected-(U1-Pad45) -> I2C_SCL
- U1 pad 46: unconnected-(U1-Pad46) -> I2C_SDA
- U1 pad 48: VDD -> +3.3V
Routing:
- net SWDIO: track 0.00 -> 13.5 mm
- net SWO: track 0.00 -> 8.01 mm
- net SWCLK: track 0.00 -> 7.86 mm
